Commit message: update camera location

File: ninjasrobot_simulation/urdf/ninjasrobot.urdf (robot description, URDF)
Before this commit: robot ninja, 6 links, 5 joints
Joints:
- joint camera_joint: origin xyz=0.215 0 0.05 rpy=0 0 0 -> xyz=0.245 0 0.05 rpy=0 0 0

Commit message: fix TF_OLD_DATA warning

File: ninjasrobot_simulation/urdf/ninjasrobot.urdf (robot description, URDF)
Before this commit: robot ninja, 6 links, 5 joints
Links:
- added link frontwhl_l_link; collision cylinder length=${wheel_width} radius=${wheel_radius}; visual cylinder length=${wheel_width} radius=${wheel_radius}
- added link frontwhl_r_link; collision cylinder length=${wheel_width} radius=${wheel_radius}; visual cylinder length=${wheel_width} radius=${wheel_radius}
Joints:
- added joint frontwhl_l_joint: type fixed, parent base_link, child frontwhl_l_link, origin xyz=${wheel_xoff} ${base_width/2+wheel_ygap} ${-wheel_zoff} rpy=0 0 0, axis 0 1 0
- added joint frontwhl_r_joint: type fixed, parent base_link, child frontwhl_r_link, origin xyz=${wheel_xoff} ${-(base_width/2+wheel_ygap)} ${-wheel_zoff} rpy=0 0 0, axis 0 1 0
